Commit message: Updated URDF so that it should now by loadable

File: collections/ur5 and objects/objects/ur5_with_gripper_description_updated/urdf/ur5.urdf (robot description, URDF)
Before this commit: robot ur5_robot, 12 links, 11 joints
Links:
- link base_link_inertia: geometry collision mesh filename=package://ur5_with_gripper_description_updated/meshes/ur5/c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; visual mesh filename=package://ur5_with_gripper_description_updated/meshes/ur5/v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
- link forearm_link: geometry collision mesh filename=package://ur5_with_gripper_description_updated/meshes/ur5/c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; visual mesh filename=package://ur5_with_gripper_description_updated/meshes/ur5/v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
- link shoulder_link: geometry collision mesh filename=package://ur5_with_gripper_description_updated/meshes/ur5/c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; visual mesh filename=package://ur5_with_gripper_description_updated/meshes/ur5/v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
- link upper_arm_link: geometry collision mesh filename=package://ur5_with_gripper_description_updated/meshes/ur5/c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; visual mesh filename=package://ur5_with_gripper_description_updated/meshes/ur5/v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
- link wrist_1_link: geometry collision mesh filename=package://ur5_with_gripper_description_updated/meshes/ur5/c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; visual mesh filename=package://ur5_with_gripper_description_updated/meshes/ur5/v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
- link wrist_2_link: geometry collision mesh filename=package://ur5_with_gripper_description_updated/meshes/ur5/c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; visual mesh filename=package://ur5_with_gripper_description_updated/meshes/ur5/v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
- link wrist_3_link: geometry collision mesh filename=package://ur5_with_gripper_description_updated/meshes/ur5/c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; visual mesh filename=package://ur5_with_gripper_description_updated/meshes/ur5/v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

Commit message: Changed ur5 updated so that it can now be loaded into the application

File: collections/ur5 and objects/objects/ur5_with_gripper_description_updated/urdf/ur5.urdf (robot description, URDF)
Before this commit: robot ur5_robot, 12 links, 11 joints
Links:
- link base_link_inertia: geometry collision mesh filename=package://ur5_with_gripper_description_updated/meshes/colli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; visual mesh filename=package://ur5_with_gripper_description_updated/meshes/visua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
- link forearm_link: geometry collision mesh filename=package://ur5_with_gripper_description_updated/meshes/colli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; visual mesh filename=package://ur5_with_gripper_description_updated/meshes/visua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
- link shoulder_link: geometry collision mesh filename=package://ur5_with_gripper_description_updated/meshes/colli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; visual mesh filename=package://ur5_with_gripper_description_updated/meshes/visua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
- link upper_arm_link: geometry collision mesh filename=package://ur5_with_gripper_description_updated/meshes/colli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; visual mesh filename=package://ur5_with_gripper_description_updated/meshes/visua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
- link wrist_1_link: geometry collision mesh filename=package://ur5_with_gripper_description_updated/meshes/colli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; visual mesh filename=package://ur5_with_gripper_description_updated/meshes/visua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
- link wrist_2_link: geometry collision mesh filename=package://ur5_with_gripper_description_updated/meshes/colli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; visual mesh filename=package://ur5_with_gripper_description_updated/meshes/visua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
- link wrist_3_link: geometry collision mesh filename=package://ur5_with_gripper_description_updated/meshes/colli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; visual mesh filename=package://ur5_with_gripper_description_updated/meshes/visua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
